File: NodePilot.kicad_sch (KiCad schematic)
At the start: 44 parts, among them K1 SRD-05VDC-SL-C, Q1 2N3904, Q2 2N2222, Q4 2N3904, T1 1:1 600R, T2 1:1 600R, U1 PC817, U2 PC817, U3 B0505S-1WR2, U4 LM358_DFN

Commit message: NodePilot PCB (#8)
NodePilot PCB
Parts:
- removed T1, T2: 1:1 600R, symbol Device:Transformer_1P_1S_SO8
- removed U4: LM358_DFN, Package_DFN_QFN:DFN-8-1EP_2x2mm_P0.5mm_EP1.05x1.75mm, symbol Amplifier_Operational:LM358_DFN
- added R15: 0 ohm, Resistor_THT:R_Axial_DIN0204_L3.6mm_D1.6mm_P5.08mm_Horizontal, symbol Device:R_US
- added T1, T2: 1:1 600R, Diode_THT:Diode_Bridge_DIP-4_W7.62mm_P5.08mm, symbol Device:Transformer_1P_1S
- added U5: LM358, symbol Amplifier_Operational:LM358
- C1, C2, C3, C4, C5, C6, C8: footprint (none) -> Capacitor_THT:CP_Radial_D5.0mm_P2.50mm
- C10, C11, C7, C9: footprint (none) -> Capacitor_THT:C_Disc_D5.0mm_W2.5mm_P2.50mm
- JP1: footprint (none) -> TerminalBlock_Phoenix:TerminalBlock_Phoenix_PT-1,5-2-3.5-H_1x02_P3.50mm_Horizontal
- R1, R10, R11, R12, R13, R16, R17, R2, R3, R4, R5, R6, R7, R8, R9: footprint (none) -> Resistor_THT:R_Axial_DIN0204_L3.6mm_D1.6mm_P5.08mm_Horizontal
- RV1, RV2: footprint (none) -> Potentiometer_THT:Potentiometer_Bourns_3296W_Vertical
- U3: footprint B0505S-1WR2_MNS -> B0505S-WR1:B0505S-1WR2_MNS; symbol B0505s:B0505S-1WR2 -> B0505S-1WR2:B0505S-1WR2
Connections:
- net +5V: now also U5.8 (V+)
- net AGND1: now also R15.1, T1.1 (AA), T2.2 (AB); no longer C10.1, U1.2
- net GND1: now also U5.4 (V-)
- net RIGGND: now also T2.3 (SA)
- net S_COR: now also U5.1
- net at C1.1, R9.2: now also T1.2 (AB)
- net at C11.2, K1.4, Q1.1 (E)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: now also T1.4 (SB)
- net at R14.1, R19.2: now also U5.2 (-)
- net at C2.2: now also T2.1 (AA)
- net at RV2.2: now also T1.3 (SA)
- net at R6.1, RV1.3: now also T2.4 (SB)
- net at R18.1, R20.2: now also U5.3 (+)
- new net: C10.1, R15.2, U1.2
Other:
- moved on the sheet: R14, R18, R19, R20, R6, U3
