File: NodePilot.kicad_pcb (KiCad board)
At the start: 2 copper layers, 39 parts, among them K1 SRD-05VDC-SL-C, Q1 2N3904, Q2 2N2222, Q4 2N3904, T1 1:1 600R, T2 1:1 600R, U1 PC817, U2 PC817, U3 B0505S-1WR2

Commit message: proper footprint
Parts:
- T1, T2: footprint Transformer_THT:Transformer_Toroid_Horizontal_D10.5mm_Amidon-T37 -> Diode_THT:Diode_Bridge_DIP-4_W7.62mm_P5.08mm
- moved T1 6.61 mm to (83.2, 41.6)
- moved T2 6.61 mm to (83.2, 29.6)
- moved R9 0.72 mm to (76.0, 41.5)
Connections:
- C1 pad 1: Net-(T1-AA) -> Net-(T1-AB)
- R9 pad 2: Net-(T1-AA) -> Net-(T1-AB)
- RV2 pad 2: Net-(T1-SB) -> Net-(T1-SA)
- T1 pad 1: Net-(T1-AA) -> GROUND
- T1 pad 4: (no net) -> Net-(Q1-E)
- T2 pad 4: (no net) -> Net-(T2-SB)

Commit message: draft
Parts:
- moved R12 26.5 mm to (81.9, 55.5)
- moved Q4 26.1 mm to (87.1, 61.2)
- moved C1 25.9 mm to (92.7, 55.5)
- moved U1 25.0 mm to (61.9, 83.5)
- moved C10 25.0 mm to (56.7, 86.0)
- moved R4 25.0 mm to (46.6, 83.7)
- moved R7 25.0 mm to (73.6, 82.2)
- moved R8 25.0 mm to (73.6, 88.7)
- moved R3 24.2 mm to (83.5, 61.3)
- moved C2 23.1 mm to (94.5, 39.0)
- moved R9 22.8 mm to (97.0, 50.5)
- moved C5 22.8 mm to (72.5, 77.5)
- moved C6 22.8 mm to (64.0, 77.5)
- moved C7 22.8 mm to (56.5, 77.5)
- moved C8 22.8 mm to (69.5, 72.2)
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
Commit message: sizing
Other:
- board outline added: 100 x 60 mm
Changed lines of the file:
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@@
 		)
+	)
+	(gr_rect
+		(start 40.5 34)
+		(end 140.5 94)
+		(stroke
+			(width 0.05)
+			(type default)
+		)
+		(fill no)
+		(layer "Edge.Cuts")
 	)
 	(embedded_fonts no)

Commit message: updated
Parts:
- added REF**: TestPoint_Pad_1.5x1.5mm, TestPoint:TestPoint_Pad_1.5x1.5mm, F.Cu at (63.5, 64.0)
- added REF**: S_COR, TerminalBlock_Phoenix:TerminalBlock_Phoenix_PT-1,5-2-3.5-H_1x02_P3.50mm_Horizontal, F.Cu at (134.5, 76.0)
- added REF**: M/A, TerminalBlock_Phoenix:TerminalBlock_Phoenix_PT-1,5-2-3.5-H_1x02_P3.50mm_Horizontal, F.Cu at (134.5, 41.0)
- added REF**: GND/PTT, TerminalBlock_Phoenix:TerminalBlock_Phoenix_PT-1,5-2-3.5-H_1x02_P3.50mm_Horizontal, F.Cu at (134.5, 84.5)
- moved R16 2.55 mm to (124.5, 66.0)
- moved JP1 1.53 mm to (134.5, 59.0)
- moved R1 1.06 mm to (128.5, 66.0), turned to -90 degrees
- moved R17 1.05 mm to (126.5, 58.9)

Commit message: updated
Parts:
- removed the REF** at (63.5, 64.0)
- moved C9 21.4 mm to (81.0, 65.2)
- moved C7 18.7 mm to (75.0, 74.5)
- moved C8 17.5 mm to (86.5, 68.0)
- moved C6 16.8 mm to (80.5, 74.5)
- moved C5 14.3 mm to (86.5, 74.5)
- moved R7 14.3 mm to (87.4, 78.5)
- moved R11 14.2 mm to (100.5, 63.5)
- moved R5 14.1 mm to (123.4, 84.5)
- moved R4 14.0 mm to (60.2, 80.5)
- moved U3 13.5 mm to (91.8, 66.2)
- moved C10 12.0 mm to (68.3, 83.0)
- moved U1 10.3 mm to (71.7, 80.5)
- moved R8 9.30 mm to (81.9, 84.5)
- moved R17 8.80 mm to (134.5, 62.5), turned to 180 degrees
- moved D3 7.81 mm to (99.5, 73.5)
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Other:
- board size 100 x 60 mm -> 100 x 55 mm

Commit message: draft 1
Parts:
- added ?: LOGO, logo:node_pilot_logo, F.Cu at (91.5, 46.0)
- moved C3 2.50 mm to (126.0, 41.5)
- moved R16 2.50 mm to (126.5, 62.4)
- moved R3 1.17 mm to (86.5, 58.0), turned to -90 degrees
- moved D3 0.69 mm to (99.5, 74.2)
- moved R8 0.50 mm to (81.9, 84.0)
- turned R1 to 0 degrees
- renumbered REF** to ?
Connections:
- ? pad 2: (no net) -> EXT_COR
- ? pad 1: (no net) -> RIGAF
- ? pad 2: (no net) -> RIGMICIN
- ? pad 1: (no net) -> PTT
- ? pad 2: (no net) -> RIGGND
Routing:
- net RIGGND: track 0.00 -> 100.2 mm
- net GROUND: track 0.00 -> 85.0 mm
- net Net-(Q2-E): track 0.00 -> 55.0 mm
- net Net-(Q1-E): track 0.00 -> 49.0 mm
- net Net-(D3-K): track 0.00 -> 41.9 mm
- net USBPWR: track 0.00 -> 19.8 mm
- net RIGAF: track 0.00 -> 18.8 mm
- net Net-(D3-A): track 0.00 -> 15.9 mm
- net Net-(Q4-C): track 0.00 -> 15.3 mm
- net Net-(Q1-B): track 0.00 -> 14.7 mm
- net Net-(T1-SA): track 0.00 -> 9.07 mm
- net Net-(R7-Pad1): track 0.00 -> 8.93 mm
- net Net-(T1-AB): track 0.00 -> 8.71 mm
- net Net-(T2-SB): track 0.00 -> 8.00 mm
- net EXT_COR: track 0.00 -> 7.61 mm
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
Commit message: draft 1
Routing:
- net RIGGND: track 100.2 -> 97.3 mm
- net Net-(Q2-E): track 55.0 -> 53.8 mm
Changed lines of the file:
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@@
 	)
 	(segment
-		(start 88.57 78.976346)
-		(end 88.57 76.02)
+		(start 86.566346 76.02)
+		(end 88.57 78.023654)
 		(width 0.5)
 		(layer "F.Cu")
@@
 	)
 	(segment
+		(start 88.57 78.023654)
+		(end 88.57 78.976346)
+		(width 0.5)
+		(layer "F.Cu")
+		(net "Net-(Q2-E)")
+	)
+	(segment
 		(start 75.73 71.27)
 		(end 75 72)
@@
 	)
 	(segment
-		(start 88.57 76.02)
-		(end 74.752233 76.02)
-		(width 0.5)
-		(layer "F.Cu")
-		(net "Net-(Q2-E)")
-	)
-	(segment
 		(start 94.92 85.54)
 		(end 94.96 85.5)
@@
 	)
 	(segment
+		(start 74.752233 76.02)
+		(end 86.566346 76.02)
+		(width 0.5)
+		(layer "F.Cu")
+		(net "Net-(Q2-E)")
+	)
+	(segment
 		(start 73.75 73.25)
 		(end 75 72)
@@
 	)
 	(segment
+		(start 103.35 78.45)
+		(end 114 78.45)
+		(width 0.5)
+		(layer "F.Cu")
+		(net "RIGGND")
+	)
+	(segment
+		(start 110 50.54)
+		(end 110 73)
+		(width 0.5)
+		(layer "F.Cu")
+		(net "RIGGND")
+	)
+	(segment
 		(start 101 86.5)
 		(end 109.45 86.5)
@@
 	)
 	(segment
-		(start 113 47.54)
-		(end 113 44)
-		(width 0.5)
-		(layer "F.Cu")
-		(net "RIGGND")
-	)
-	(segment
-		(start 103.35 78.45)
+		(start 109.45 86.5)
+		(end 114 81.95)
+		(width 0.5)
+		(layer "F.Cu")
+		(net "RIGGND")
+	)
+	(segment
+		(start 114 81.95)
+		(end 114 78.45)
+		(width 0.5)
+		(layer "F.Cu")
+		(net "RIGGND")
+	)
+	(segment
+		(start 114 77)
+		(end 114 78.45)
+		(width 0.5)
+		(layer "F.Cu")
+		(net "RIGGND")
+	)
+	(segment
+		(start 114 78.45)
 		(end 117.5 78.45)
-		(width 0.5)
-		(layer "F.Cu")
-		(net "RIGGND")
-	)
-	(segment
-		(start 110 70.95)
-		(end 117.5 78.45)
-		(width 0.5)
-		(layer "F.Cu")
-		(net "RIGGND")
-	)
-	(segment
-		(start 110 50.54)
-		(end 110 70.95)
 		(width 0.5)
 		(layer "F.Cu")
@@
 	)
 	(segment
+		(start 110 73)
+		(end 114 77)
+		(width 0.5)
+		(layer "F.Cu")
+		(net "RIGGND")
+	)
+	(segment
 		(start 113 44)
 		(end 121 44)
@@
 	)
 	(segment
-		(start 109.45 86.5)
-		(end 117.5 78.45)
-		(width 0.5)
-		(layer "F.Cu")
-		(net "RIGGND")
-	)
-	(segment
 		(start 100.04 85.5)
 		(end 100.59 86.05)
@@
 	)
 	(segment
+		(start 113 47.54)
+		(end 110 50.54)
+		(width 0.5)
+		(layer "F.Cu")
+		(net "RIGGND")
+	)
+	(segment
 		(start 117.5 78.45)
 		(end 123.95 78.45)
@@
 	)
 	(segment
-		(start 110 50.54)
+		(start 113 44)
 		(end 113 47.54)
 		(width 0.5)

Commit message: super update
Parts:
- added ?: COS, TestPoint:TestPoint_Pad_1.5x1.5mm, F.Cu at (92.0, 47.0)
- added ?: GND, TestPoint:TestPoint_Pad_1.5x1.5mm, F.Cu at (92.0, 49.5)
- added ?: PTT, TestPoint:TestPoint_Pad_1.5x1.5mm, F.Cu at (92.0, 39.5)
- added ?: MIC, TestPoint:TestPoint_Pad_1.5x1.5mm, F.Cu at (92.0, 44.5)
- added ?: SPK, TestPoint:TestPoint_Pad_1.5x1.5mm, F.Cu at (92.0, 37.0)
- added ?: PWR, TestPoint:TestPoint_Pad_1.5x1.5mm, F.Cu at (92.0, 42.0)
- added R15: 0 ohm, Resistor_THT:R_Axial_DIN0204_L3.6mm_D1.6mm_P5.08mm_Horizontal, F.Cu at (76.0, 63.4)
- ?: value M/A -> AF-MIC
- ?: value GND/PTT -> PTT-GND
- JP1: value Jumper JP1 -> JP1
- moved R4 13.0 mm to (70.5, 72.5), turned to -90 degrees
- moved ? 9.29 mm to (82.5, 48.5), turned to -90 degrees
Connections:
- C10 pad 1: GROUND -> Net-(C10-Pad1)
- U1 pad 2: GROUND -> Net-(C10-Pad1)
Routing:
- net GPIO3: track 0.00 -> 42.7 mm
- net USBPWR: track 19.8 -> 58.9 mm
- net Net-(C10-Pad1): track 0.00 -> 20.5 mm
- net VOLDN: track 4.93 -> 18.2 mm
- net MICIN: track 0.00 -> 13.0 mm
- net GROUND: track 85.0 -> 73.6 mm
- net LOL: track 0.00 -> 7.83 mm
